File: LO-test-board.kicad_sch (KiCad schematic)
At the start: 122 parts, among them J1 RF_OUT, J3 RF_OUT, J5 TEST, J6 TEST, J7 Conn_01x08, U12 GALI-39, U15 PAT1220-C-3DB, U17 TLV1117LV-33, U18 TLV1117LV-18, U2 LM7805_TO220, U3 MTX2-143+, U4 AVA-183A+, X1 ASCO

Commit message: updated schematic pdf
Other:
- company: (none) -> Max Xiang
- title: (none) -> STuW81300 TEST BOARD
Changed lines of the file:
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@@
 	(generator_version "9.0")
 	(paper "A2")
+	(title_block
+		(title "STuW81300 TEST BOARD")
+		(date "2025-06-28")
+		(company "Max Xiang")
+	)
 	(text "STuW81300 uses SPI mode 3."
 		(exclude_from_sim no)
